File: USB_Hub.kicad_sch (KiCad schematic)
At the start: 53 parts, among them J12 USB4105-GF-A-120, U1 USB2514B_Bi, U2 MIC2026-1xM, U3 MIC2026-1xM, U8 USBLC6-2SC6, U9 AMS1117-3.3, Y1 Crystal_GND24

Commit message: final
Other:
- note added: "LDO"
- note added: "Power Switches"
- note added: "USB HUB"
- moved on the sheet: C1, C10, C11, C12, C13, C14, C15, C16, C17, C18, C19, C2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
